File: Controlador CC-20A/PCB1/Controlador_CC_20A.kicad_pcb (KiCad board)
At the start: 2 copper layers, 48 x 48 mm, 13 parts, among them J1 Conn_01x02, J2 Conn_01x02, J3 Conn_01x02, Q1 IRLZ44N, U1 4N25

Commit message: Diseño de PCB V1.
Parts:
- J2, J3: value Conn_01x02 -> Screw_Terminal_01x02; footprint TerminalBlock_MetzConnect:TerminalBlock_MetzConnect_Type094_RT03502HBLU_1x02_P5.00mm_Horizontal -> TerminalBlock_Phoenix:TerminalBlock_Phoenix_MKDS-1,5-2-5.08_1x02_P5.08mm_Horizontal
- moved HS2 1.83 mm to (154.0, 93.9)
- moved Q1 1.55 mm to (149.7, 91.3)
- moved J3 1.10 mm to (170.0, 100.2)
- moved D2 0.99 mm to (168.3, 94.1)
- moved R2 0.91 mm to (143.1, 108.3)
- moved J2 0.45 mm to (170.0, 82.5)
Routing:
- net /Salida: track 32.4 -> 42.4 mm
- net /VCC: track 69.2 -> 59.9 mm
- net GNDPWR: track 66.1 -> 67.6 mm
Other:
- board text added: "Controlador PWM 20A - V1 2025"
- board text added: "SCA-UNDAV (ARG) UNIVERSIDAD PUBLICA"
- board text removed: "Controlador PWM 10A 24V - V1 2025"
- board text removed: "HECHO EN ARGENTINA UNDAV-SCA"
